File: max2771.kicad_sch (KiCad schematic)
At the start: 20 parts, among them U1 MAX2771ETI+

Commit message: finished v1
Parts:
- added C2: 10nF, Capacitor_SMD:C_0603_1608Metric, symbol Device:C_Small
- C0, C1, C11, C12: value C_Small -> 0.47nF; footprint (none) -> Capacitor_SMD:C_0603_1608Metric
- C10, C13, C4, C7, C8, C9: value C_Small -> 0.1μF; footprint (none) -> Capacitor_SMD:C_0603_1608Metric
- C14: value C_Small -> 0.1nF; footprint (none) -> Capacitor_SMD:C_0603_1608Metric
- C15: value C_Small -> 1.7 pF; footprint (none) -> Capacitor_SMD:C_0603_1608Metric
- C16: value C_Small -> 1.1 pF; footprint (none) -> Capacitor_SMD:C_0603_1608Metric
- C3: value C_Small -> 10nF; footprint (none) -> Capacitor_SMD:C_0603_1608Metric
- C5: value C_Small -> 0.75nF; footprint (none) -> Capacitor_SMD:C_0603_1608Metric
- C6: value C_Small -> 15pF; footprint (none) -> Capacitor_SMD:C_0603_1608Metric
- L0: value L -> 5.6 nH; footprint (none) -> Inductor_SMD:L_1206_3216Metric
- L1: value L -> 8.4 nH; footprint (none) -> Inductor_SMD:L_1206_3216Metric
- R0: value R_US -> 15k; footprint (none) -> Resistor_SMD:R_0805_2012Metric
- U1: footprint 21-0140L_T2855-8_MXM -> footprints:21-0140L_T2855-8_MXM
Connections:
- net REF_CLK_OUT: now also C2.2; no longer U1.4 (CLKOUT)
- new net: C2.1, U1.4 (CLKOUT)
Other:
- company: (none) -> K. Karpacz
