File: max2771eval.kicad_pcb (KiCad board)
At the start: 4 copper layers, 95 x 80.6 mm, 72 parts, among them IC2 MAX8510EXK33+T, IC3 MAX8510EXK33+T, IC4 MAX8510EXK33+T, J1 Conn_Coaxial, J2 Conn_Coaxial, J4 Conn_02x07_Odd_Even, J5 Conn_01x05_Socket, U1 MAX2771ETI+, U2 YAAJ_BluePill_SWD_Breakout, X1 16.368MHz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

Commit message: outputs
Changed lines of the file:
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@@
 		(tenting front back)
 		(pcbplotparams
-			(layerselection 0x00000000_00000000_55555555_5755f5ff)
+			(layerselection 0x00000000_00000000_55555555_55555555)
 			(plot_on_all_layers_selection 0x00000000_00000000_00000000_00000000)
 			(disableapertmacros no)
@@
 			(pdf_back_fp_property_popups yes)
 			(pdf_metadata yes)
-			(pdf_single_document no)
+			(pdf_single_document yes)
 			(dxfpolygonmode yes)
 			(dxfimperialunits yes)
@@
 			(psnegative no)
 			(psa4output no)
-			(plot_black_and_white yes)
+			(plot_black_and_white no)
 			(plotinvisibletext no)
 			(sketchpadsonfab no)
@@
 			(crossoutdnponfab yes)
 			(subtractmaskfromsilk no)
-			(outputformat 1)
+			(outputformat 4)
 			(mirror no)
-			(drillshape 1)
+			(drillshape 0)
 			(scaleselection 1)
-			(outputdirectory "")
+			(outputdirectory "plots2")
 		)
 	)
@@
 		)
 		(fp_text user "*"
-			(at -3.5 -2.31972 180)
+			(at -3.7 -2.2 180)
 			(unlocked yes)
 			(layer "F.SilkS")
@@
 			)
 		)
-		(fp_text user "${REFERENCE}"
-			(at 0 0 180)
+		(fp_text user "*"
+			(at -1.8923 -1.75 180)
 			(unlocked yes)
 			(layer "F.Fab")
@@
 			)
 		)
-		(fp_text user "*"
-			(at -1.8923 -1.75 0)
+		(fp_text user "${REFERENCE}"
+			(at 0 0 180)
+			(unlocked yes)
 			(layer "F.Fab")
 			(effects
@@
 		)
 		(embedded_fonts no)
+		(model "${KIPRJMOD}/lib/ul_MAX2771ETI-/21-0140L_T2855-8_MXM.step"
+			(offset
+				(xyz 0 0 0)
+			)
+			(scale
+				(xyz 1 1 1)
+			)
+			(rotate
+				(xyz 0 0 0)
+			)
+		)
 	)
 	(footprint "Capacitor_SMD:C_0603_1608Metric"
