File: max2771eval.kicad_sch (KiCad schematic)
At the start: 0 parts

Commit message: finished v1
Parts:
- added C35: 10nF, Capacitor_SMD:C_0603_1608Metric, symbol Device:C_Small
- added D2, D3, D4: LED, Diode_SMD:D_0805_2012Metric, symbol Device:LED
- added H1, H2, H3: MountingHole_Pad, MountingHole:MountingHole_2.2mm_M2_Pad_Via, symbol Mechanical:MountingHole_Pad
- added J1, J2: Conn_Coaxial, Connector_Coaxial:SMA_Amphenol_901-143_Horizontal, symbol Connector:Conn_Coaxial
- added J4: Conn_02x07_Odd_Even, Connector_PinSocket_2.54mm:PinSocket_2x07_P2.54mm_Vertical, symbol Connector_Generic:Conn_02x07_Odd_Even
- added J5: Conn_01x05_Socket, Connector_PinSocket_2.54mm:PinSocket_1x05_P2.54mm_Vertical, symbol Connector:Conn_01x05_Socket
- added JP1, JP4: Jumper_3_Bridged12, Connector_PinHeader_2.54mm:PinHeader_1x03_P2.54mm_Vertical, symbol Jumper:Jumper_3_Bridged12
- added JP2, JP3: Jumper_2_Bridged, Connector_PinHeader_2.54mm:PinHeader_1x02_P2.54mm_Vertical, symbol Jumper:Jumper_2_Bridged
- added JP5: Jumper_2_Open, Connector_PinHeader_2.54mm:PinHeader_1x02_P2.54mm_Vertical, symbol Jumper:Jumper_2_Open
- added L4, L5: 5.6nH, Inductor_SMD:L_1206_3216Metric, symbol Device:L_Ferrite
- added R20, R21, R22: 1k, Resistor_SMD:R_0805_2012Metric, symbol Device:R_US
- added R23: 25k, Resistor_SMD:R_0805_2012Metric, symbol Device:R_US
- added TP4: ADC_CLK_EXT, TestPoint:TestPoint_Pad_D1.5mm, symbol Connector:TestPoint
- added TP5: REF_CLK, TestPoint:TestPoint_Pad_D1.5mm, symbol Connector:TestPoint
- added U2: YAAJ_BluePill_SWD_Breakout, BluePill:YAAJ_BluePill_SWD_1, symbol YAAJ_BluePill_SWD_Breakout:YAAJ_BluePill_SWD_Breakout
- added X1: 16.368MHz, PCM_Crystal_AKL:Crystal_SMD_5032-4Pin_5.0x3.2mm, symbol PCM_Crystal_AKL:SMD5032-4
- added Y1: ATX-H11-F-24.000MHz-F25-T, ATX-H11-F-24.000MHz-F25-T:ATXH11F24000MHzF25T, symbol ATX-H11-F-24_000MHz-F25-T:ATX-H11-F-24.000MHz-F25-T
Connections:
- new net: D4.2 (A), U2.16 (PB8)
- new net: JP5.2 (B), R23.1, Y1.1 (~{INH})
- new net: JP1.1 (A), Y1.3 (OUTPUT)
- new net: D3.1 (K), R21.2
- new net: D4.1 (K), R22.2
- new net: JP1.3 (B), X1.3
- new net: JP3.1 (A), L5.1
- new net: JP2.1 (A), L4.1
- new net: D2.1 (K), R20.2
- new net +3.3V_IO: C35.2, R23.2, Y1.4 (VDD)
- new net +3.3_ANT: JP2.2 (B), JP3.2 (B)
- new net +5V_USB: U2.18 (5V)
- new net ADC_CLK_A: J4.9 (Pin_9), JP4.2 (C)
- new net ADC_CLK_A_EXT: J4.13 (Pin_13), JP4.3 (B), TP4.1
- new net A_CSN: J5.3 (Pin_3), U2.29 (PA4)
- new net A_I0: J4.1 (Pin_1)
- new net A_I1: J4.5 (Pin_5)
- new net A_LOCK_DETECT: D2.2 (A), J4.11 (Pin_11), U2.34 (PB1)
- new net A_Q0: J4.3 (Pin_3)
- new net A_Q1: J4.7 (Pin_7)
- new net A_SCLK: J5.1 (Pin_1), U2.30 (PA5)
- new net A_SDATA: J5.2 (Pin_2), U2.32 (PA7)
- new net A_SHDN: D3.2 (A), J5.4 (Pin_4), U2.33 (PB0)
- new net GND: C35.1, H1.1, H2.1, H3.1, J1.2 (Ext), J2.2 (Ext), J4.10 (Pin_10), J4.12 (Pin_12), J4.14 (Pin_14), J4.2 (Pin_2), J4.4 (Pin_4), J4.6 (Pin_6), J4.8 (Pin_8), J5.5 (Pin_5), JP5.1 (A), R20.1, R21.1, R22.1, U2.19 (GND), U2.39 (GND), U2.40 (GND), U2.41 (GND), X1.1, X1.2, X1.4, Y1.2 (GND)
- new net REF_CLK_A: JP1.2 (C)
- new net REF_CLK_OUT_A: JP4.1 (A), TP5.1
- new net RF_HIGH_BAND_IN_A: J2.1 (In), L5.2
- new net RF_LOW_BAND_IN_A: J1.1 (In), L4.2
Other:
- added sheet Power (power.kicad_sch)
- sheet max2771 ports: added ADC_CLKIN, CSN, LD, REF_CLK, REF_CLK_OUT, RF_HI_IN, RF_LO_IN, SCLK, SDATA, SHDN, VCCADC, VCCCP, VCCD, VCCIF, VCC_RF, VCC_VCO; removed none
- note added: "close when using XTAL"
- company: (none) -> K. Karpacz
- title: (none) -> MAX2771 test board

Commit message: outputs
Parts:
- L4, L5: value 5.6nH -> 1uH
- TP4, TP5: now left out of the parts list
Changed lines of the file:
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@@
 		(unit 1)
 		(exclude_from_sim no)
-		(in_bom yes)
+		(in_bom no)
 		(on_board yes)
 		(dnp no)
@@
 		(unit 1)
 		(exclude_from_sim no)
-		(in_bom yes)
+		(in_bom no)
 		(on_board yes)
 		(dnp no)
@@
 			)
 		)
-		(property "Value" "5.6nH"
+		(property "Value" "1uH"
 			(at 60.96 71.1199 0)
 			(effects
@@
 			)
 		)
-		(property "Value" "5.6nH"
+		(property "Value" "1uH"
 			(at 60.96 49.5299 0)
 			(effects
