File: power.kicad_sch (KiCad schematic)
At the start: 24 parts, among them IC2 MAX8510EXK33+T, IC3 MAX8510EXK33+T, IC4 MAX8510EXK33+T

Commit message: outputs
Parts:
- TP1, TP2, TP3: now left out of the parts list
Changed lines of the file:
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@@
 		(unit 1)
 		(exclude_from_sim no)
-		(in_bom yes)
+		(in_bom no)
 		(on_board yes)
 		(dnp no)
@@
 		(unit 1)
 		(exclude_from_sim no)
-		(in_bom yes)
+		(in_bom no)
 		(on_board yes)
 		(dnp no)
@@
 		(unit 1)
 		(exclude_from_sim no)
-		(in_bom yes)
-		(on_board yes)
-		(dnp no)
+		(in_bom no)
+		(on_board yes)
+		(dnp no)
